File: Hardware/kicad/CANNode/CANNode.kicad_pcb (KiCad board)
At the start: 2 copper layers, 55 parts, among them J1 Conn_01x04, J11 Conn_01x04, J12 Conn_01x04, J2 Conn_01x04, J21 Conn_01x04, J31 Conn_01x04, J41 Conn_01x04, J42 Conn_01x04, J43 Conn_01x04, J44 Conn_01x04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

Commit message: kicad 101
Parts:
- removed C11: C, Capacitor_SMD:C_0805_2012Metric_Pad1.15x1.40mm_HandSolder
- removed JP11, JP12: Jumper_NC_Small, Jumper:SolderJumper-2_P1.3mm_Open_RoundedPad1.0x1.5mm
- removed JP42, JP43, JP44: Jumper_3_Bridged12, Jumper:SolderJumper-3_P1.3mm_Bridged2Bar12_RoundedPad1.0x1.5mm_NumberLabels
- added REF**: MountingHole_2.2mm_M2_DIN965, MountingHole:MountingHole_2.2mm_M2_DIN965, F.Cu at (72.8, 91.7)
- added REF**: MountingHole_2.2mm_M2_DIN965, MountingHole:MountingHole_2.2mm_M2_DIN965, F.Cu at (133.8, 39.2)
- added REF**: MountingHole_2.2mm_M2_DIN965, MountingHole:MountingHole_2.2mm_M2_DIN965, F.Cu at (133.8, 91.7)
- added REF**: MountingHole_2.2mm_M2_DIN965, MountingHole:MountingHole_2.2mm_M2_DIN965, F.Cu at (72.8, 39.2)
- C3, C4, JP31, JP41, R11, R12, R2, R21, R22, R24, R25, R3, R4, R5, R6, U41: moved to B.Cu
- J12: footprint CANNode:OWN_KF141V-P4_simple -> Connector_PinHeader_2.54mm:PinHeader_1x04_P2.54mm_Vertical
- U2: moved to F.Cu
- moved JP31 119.5 mm to (76.6, 52.8)
- moved R6 109.0 mm to (79.4, 43.9), turned to 180 degrees
- moved J41 108.3 mm to (108.6, 43.2), turned to 180 degrees
- moved C5 104.8 mm to (76.8, 55.9)
- moved U31 102.7 mm to (79.4, 64.5), turned to 90 degrees
- moved C4 97.0 mm to (92.1, 51.8), turned to 180 degrees
- moved R1 92.8 mm to (82.2, 77.2)
- moved J42 92.6 mm to (122.6, 41.9), turned to 0 degrees
- moved R11 91.4 mm to (88.3, 45.7), turned to 90 degrees
- moved C7 91.1 mm to (84.5, 68.6), turned to 270 degrees
- moved C8 88.9 mm to (83.4, 64.5), turned to 90 degrees
- moved J91 88.6 mm to (128.9, 78.7), turned to 90 degrees
- moved J43 87.4 mm to (130.2, 41.9), turned to 0 degrees
- moved R12 87.0 mm to (98.4, 45.7), turned to 180 degrees
- moved JP1 86.6 mm to (78.4, 77.2), turned to 270 degrees
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Connections:
- net Net-(J31-Pad2) renamed /UA1+
- net Net-(J31-Pad3) renamed /UA1-
- net Net-(J42-Pad2) renamed /D2-
- net Net-(J43-Pad2) renamed /D3-
- net Net-(J44-Pad2) renamed /D4-
- net Net-(U1-Pad10) renamed /DI2_8
- net Net-(U1-Pad11) renamed /EN34_9
- net Net-(U1-Pad3) renamed /TX2
- net Net-(U1-Pad4) renamed /UA3EN_2
- C7 pad 1: +5V -> +3V3
- C8 pad 1: +5V -> +3V3
- C9 pad 1: +5V -> +3V3
- J1 pad 2: /CAN- -> /CAN+
- J1 pad 3: /CAN+ -> /CAN-
- J11 pad 4: Net-(J11-Pad4) -> +12V
- J12 pad 4: Net-(J12-Pad4) -> +12V
- J2 pad 2: /CAN- -> /CAN+
- J2 pad 3: /CAN+ -> /CAN-
- J42 pad 4: Net-(J42-Pad4) -> +5V
- J43 pad 4: Net-(J43-Pad4) -> +5V
- J44 pad 4: Net-(J44-Pad4) -> +5V
- J81 pad 2: /6 -> /10
- J81 pad 3: /10 -> /6
- JP1 pad 2: /CAN- -> /CAN+
- JP22 pad 1: Net-(J61-Pad7) -> Net-(JP22-Pad1)
- JP22 pad 2: Net-(JP22-Pad2) -> Net-(J61-Pad7)
- R1 pad 2: /CAN+ -> /CAN-
- R22 pad 1: Net-(JP22-Pad2) -> Net-(JP22-Pad1)
- U21 pad 4: Net-(JP22-Pad2) -> Net-(JP22-Pad1)
Routing:
- net /CAN+: track 0.00 -> 48.2 mm, vias 0 -> 1
- net /CAN-: track 0.00 -> 42.6 mm, vias 0 -> 1
- net +5V: track 0.00 -> 41.0 mm
- net /DI2_8: track 0.00 -> 32.8 mm
- net /DI1_7: track 0.00 -> 28.3 mm
- net /SCL0_16: track 0.00 -> 24.0 mm
- net /EN34_9: track 0.00 -> 23.6 mm
- net /D4-: track 0.00 -> 22.3 mm
- net /D3-: track 0.00 -> 21.8 mm
- net Net-(J61-Pad7): track 0.00 -> 21.5 mm
- net /D3+: track 0.00 -> 20.4 mm
- net +3V3: track 0.00 -> 19.4 mm, vias 0 -> 1
- net /D4+: track 0.00 -> 19.0 mm
- net GND: track 0.00 -> 18.8 mm, vias 0 -> 16
- net Net-(JP22-Pad1): track 0.00 -> 16.3 mm
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- added copper zone on In1.Cu, net GND
Other:
- board outline added: 66 x 57.5 mm
- copper layers 2 -> 4
- net class Default: clearance 0.2 -> 0.175; trace_width 0.25 -> 0.3; via_dia 0.8 -> 0.6858; via_drill 0.4 -> 0.3302
- net class Power added: clearance 0.2, trace_width 0.5, via_dia 1.25, via_drill 0.5
- rule trace_clearance: 0.2 -> 0.175
- rule trace_min: 0.2 -> 0.1524
- rule via_min_drill: 0.3 -> 0.3302
- rule via_min_size: 0.4 -> 0.6858
