File: Hardware/kicad/CANNode.kicad_pcb (KiCad board)
At the start: 4 copper layers, 66.5 x 57 mm, 58 parts, among them J1 Conn_01x04, J11 Conn_01x04, J12 Conn_01x04, J2 Conn_01x04, J21 Conn_01x04, J31 Conn_01x04, J41 Conn_01x04, J42 Conn_01x04, J43 Conn_01x04, J44 Conn_01x04, J61 Conn_02x04_Odd_Even, J81 Conn_01x10, J91 Conn_01x04, U1 Teensy3.2, U2 SN65HVD230, U21 PCA9306, U31 MAX3485, U41 MAX3485, U91 LM1117-5.0

Commit message: First current messurement attempts
Parts:
- removed ? (x2): , own:LOGO_MID
- removed the C1 at (104.1, 83.8) (x2)
- removed the C2 at (118.1, 83.8) (x2)
- removed J91: Conn_01x04, CANNode:OWN_KF141V-P4_simple
- removed REF** (x5): MountingHole_2.5mm, MountingHole:MountingHole_2.5mm
- removed REF**: KiCAD Logo, Symbol:Symbol_KiCAD-Logo_CopperAndSilkScreenTop
- removed REF**: OSHW-Symbol_6.7x6mm_SilkScreen, Symbol:OSHW-Symbol_6.7x6mm_SilkScreen
- removed the U1 at (93.3, 66.0)
- removed U91: LM1117-5.0, Package_TO_SOT_SMD:SOT-223-3_TabPin2
- added C10: 100n, Capacitor_SMD:C_0805_2012Metric_Pad1.15x1.40mm_HandSolder, B.Cu at (106.3, 84.6)
- added C11: 100n, Capacitor_SMD:C_0805_2012Metric_Pad1.15x1.40mm_HandSolder, B.Cu at (110.6, 80.5)
- added C12: 100n, Capacitor_SMD:C_0805_2012Metric_Pad1.15x1.40mm_HandSolder, B.Cu at (114.7, 84.7)
- added C9: C, Capacitor_SMD:C_0805_2012Metric_Pad1.15x1.40mm_HandSolder, F.Cu at (140.8, 92.7)
- added J13: Conn_01x04, CANNode:OWN_KF141V-P4_simple, F.Cu at (128.9, 78.1)
- added R12: 0R1, Resistor_SMD:R_2512_6332Metric, F.Cu at (105.8, 84.7)
- added R15: 10, Resistor_SMD:R_0805_2012Metric_Pad1.15x1.40mm_HandSolder, F.Cu at (97.7, 78.2)
- added R16: 10, Resistor_SMD:R_0805_2012Metric_Pad1.15x1.40mm_HandSolder, F.Cu at (108.8, 82.7)
- added R17: 0R1, Resistor_SMD:R_2512_6332Metric, F.Cu at (91.8, 77.2)
- added R18: 10, Resistor_SMD:R_0805_2012Metric_Pad1.15x1.40mm_HandSolder, F.Cu at (108.8, 86.6)
- added R19: 10, Resistor_SMD:R_0805_2012Metric_Pad1.15x1.40mm_HandSolder, F.Cu at (97.7, 76.2)
- added R20: 0R1, Resistor_SMD:R_2512_6332Metric, F.Cu at (115.3, 84.7)
- added R21: 10, Resistor_SMD:R_0805_2012Metric_Pad1.15x1.40mm_HandSolder, F.Cu at (112.4, 86.7)
- added R22: 10, Resistor_SMD:R_0805_2012Metric_Pad1.15x1.40mm_HandSolder, F.Cu at (112.4, 82.8)
- added U3: Teensy3.2, teensy:Teensy3_min, F.Cu at (93.3, 66.0)
- added U6: INA3221, Package_DFN_QFN:QFN-16-1EP_4x4mm_P0.65mm_EP2.1x2.1mm, B.Cu at (110.6, 84.6)
- MOD1: value OWN_DCDC -> DSN-MINI-360; moved to B.Cu
- U4: renamed from U41; value MAX3485 -> MAX3032
- moved MOD1 16.2 mm to (133.6, 96.6)
- renumbered C3 to C1, C4 to C2, C5 to C3, C6 to C4, C7 to C5, C8 to C6, C9 to C7, C10 to C8, J12 to J10, J44 to J11, J21 to J12, J31 to J3, J81 to J4, J41 to J5, J61 to J6, J42 to J7, J11 to J8, J43 to J9, JP31 to JP1, JP1 to JP2, JP41 to JP3, JP21 to JP4, R6 to R1, R24 to R10, R25 to R11, R22 to R13, R21 to R14, R1 to R2, R2 to R3, R11 to R5, R12 to R6, R3 to R7, R5 to R8, R23 to R9, U31 to U1, U21 to U5
Connections:
- net Net-(J12-Pad2) renamed /OW15
- J1 pad 4: +12V -> +12LF
- J4 pad 4: /16 -> /18
- J4 pad 5: /17 -> /19
- MOD1 pad IN+: +12V -> (no net)
- MOD1 pad OUT+: +5V -> (no net)
- U2 pad 5: Net-(U2-Pad5) -> (no net)
Routing:
- net +12V: track 134.3 -> 94.7 mm, vias 9 -> 2
- net +5V: track 46.3 -> 34.7 mm, vias 8 -> 3
- net Net-(C12-Pad2): track 0.00 -> 5.56 mm, vias 0 -> 1
- net Net-(C12-Pad1): track 0.00 -> 5.05 mm, vias 0 -> 1
- net /19: track 0.00 -> 3.81 mm
- net /18: track 0.00 -> 3.81 mm
- net /17: track 3.81 -> 0.00 mm
- net /16: track 3.81 -> 0.00 mm
- net +5P: track 0.00 -> 3.09 mm
- net Net-(C10-Pad1): track 0.00 -> 2.95 mm, vias 0 -> 1
- net Net-(C10-Pad2): track 0.00 -> 2.39 mm
- net GND: vias 26 -> 7
- removed copper zone on In2.Cu, net +12V
