File: Hardware/kicad/CANNode.sch (KiCad schematic (older format))
At the start: 49 parts, among them J1 Conn_01x04, J11 Conn_01x04, J12 Conn_01x04, J2 Conn_01x04, J21 Conn_01x04, J31 Conn_01x04, J41 Conn_01x04, J42 Conn_01x04, J43 Conn_01x04, J44 Conn_01x04, J51 Conn_01x02, J61 Conn_02x04_Odd_Even, J81 Conn_01x10, J91 Conn_01x04, U1 Teensy3.2, U2 SN65HVD230, U21 PCA9306, U31 MAX3485, U41 MAX3485, U91 LM1117-5.0

Commit message: late changes
Parts:
- removed J51: Conn_01x02, Connector_PinHeader_2.54mm:PinHeader_1x02_P2.54mm_Vertical, symbol Connector_Generic:Conn_01x02
- removed JP21, JP22: Jumper_NC_Small, Connector_PinHeader_2.54mm:PinHeader_1x02_P2.54mm_Vertical, symbol Device:Jumper_NC_Small
- added C11, C12: CP, Capacitor_SMD:CP_Elec_3x5.4, symbol Device:CP_Small
- added JP21: Conn_02x03_Odd_Even, Connector_PinHeader_2.54mm:PinHeader_2x03_P2.54mm_Vertical, symbol Connector_Generic:Conn_02x03_Odd_Even
- MOD1: Name (none) -> DSN-MINI-36 (LM2596)
Connections:
- wire segments 375 -> 374
Other:
- moved on the sheet: C1, C10, C2, C3, C4, C5, C6, C7, C8, C9, J1, J11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

Commit message: more clearance in Layer 2
Parts:
- MOD1: value OWN_DCDC -> DSN-MINI-360; symbol CANNode:OWN_DCDC -> 000_my_lib:DSN-MINI-360
- U41: symbol zzz_my_lib:MAX3032 -> 000_my_lib:MAX3032
Changed lines of the file:
@@
 $EndComp
 $Comp
-L CANNode:OWN_DCDC MOD1
+L 000_my_lib:DSN-MINI-360 MOD1
 U 1 1 5BE5A42C
-P 2650 5300
-F 0 "MOD1" H 2650 5300 45  0001 C CNN
-F 1 "OWN_DCDC" H 2650 5300 45  0001 C CNN
-F 2 "CANNode:OWN_DC-DC" H 2650 5300 50  0001 C CNN
-F 3 "" H 2650 5300 50  0001 C CNN
-F 4 "DSN-MINI-36  (LM2596)" H 2650 5300 50  0001 C CNN "Name"
-	1    2650 5300
+P 2450 5450
+F 0 "MOD1" H 2450 5450 45  0001 C CNN
+F 1 "DSN-MINI-360" H 2450 5450 45  0001 C CNN
+F 2 "CANNode:OWN_DC-DC" H 2450 5450 50  0001 C CNN
+F 3 "" H 2450 5450 50  0001 C CNN
+F 4 "DSN-MINI-36  (LM2596)" H 2450 5450 50  0001 C CNN "Name"
+	1    2450 5450
 	1    0    0    -1
 $EndComp
@@
 	2200 5200 2200 5100
 Wire Wire Line
-	2250 5200 2200 5200
-Wire Wire Line
-	2250 5400 2200 5400
-Wire Wire Line
 	2200 5500 2200 5400
 Wire Wire Line
-	3050 5400 3100 5400
-Wire Wire Line
 	3100 5400 3100 5500
-Wire Wire Line
-	3050 5200 3100 5200
 Wire Wire Line
 	3100 5200 3100 5100
@@
 	5700 3300 5700 3850
 $Comp
-L zzz_my_lib:MAX3032 U41
+L 000_my_lib:MAX3032 U41
 U 1 1 5C608233
 P 2600 3350
@@
 Connection ~ 3100 5200
 Connection ~ 3100 5400
+Wire Wire Line
+	3000 5200 3100 5200
+Wire Wire Line
+	3000 5400 3100 5400
+Wire Wire Line
+	2200 5200 2350 5200
+Wire Wire Line
+	2200 5400 2350 5400
 $EndSCHEMATC

Commit message: cleanup after order
Connections:
- wire segments 374 -> 370
Other:
- moved on the sheet: R2
Changed lines of the file:
@@
 L Device:R_Small R2
 U 1 1 5C60824F
-P 1750 2600
-F 0 "R2" V 1650 2600 50  0000 C CNN
-F 1 "120" V 1855 2600 50  0000 C CNN
-F 2 "Resistor_SMD:R_0805_2012Metric_Pad1.15x1.40mm_HandSolder" H 1750 2600 50  0001 C CNN
-F 3 "~" H 1750 2600 50  0001 C CNN
-	1    1750 2600
+P 1800 2600
+F 0 "R2" V 1700 2600 50  0000 C CNN
+F 1 "120" V 1905 2600 50  0000 C CNN
+F 2 "Resistor_SMD:R_0805_2012Metric_Pad1.15x1.40mm_HandSolder" H 1800 2600 50  0001 C CNN
+F 3 "~" H 1800 2600 50  0001 C CNN
+	1    1800 2600
 	-1   0    0    1
 $EndComp
@@
 $EndComp
 Wire Wire Line
-	1550 2450 1550 2550
-Wire Wire Line
-	1550 2550 1450 2550
-Wire Wire Line
-	1550 2450 1750 2450
-Wire Wire Line
-	1450 2650 1550 2650
-Wire Wire Line
-	1550 2650 1550 2750
-Wire Wire Line
-	1550 2750 1750 2750
-Wire Wire Line
-	1750 2700 1750 2750
-Wire Wire Line
-	1750 2500 1750 2450
+	1650 2450 1650 2550
+Wire Wire Line
+	1650 2550 1450 2550
+Wire Wire Line
+	1650 2450 1800 2450
+Wire Wire Line
+	1450 2650 1650 2650
+Wire Wire Line
+	1650 2650 1650 2750
+Wire Wire Line
+	1650 2750 1800 2750
+Wire Wire Line
+	1800 2700 1800 2750
+Wire Wire Line
+	1800 2500 1800 2450
 $Comp
 L power:+12V #PWR?
@@
 	6050 5300 5400 5300
 Connection ~ 5400 5300
-Wire Wire Line
-	1750 2750 1900 2750
-Wire Wire Line
-	1900 2750 1900 2650
-Connection ~ 1750 2750
-Wire Wire Line
-	1750 2450 1900 2450
-Wire Wire Line
-	1900 2450 1900 2550
-Connection ~ 1750 2450
+Connection ~ 1800 2750
+Connection ~ 1800 2450
 Wire Wire Line
 	1800 3550 1900 3550
@@
 Text Label 3200 3200 1    50   ~ 0
 DI2_8
-Text Label 1900 2550 0    50   ~ 0
+Text Label 1900 2450 0    50   ~ 0
 D1+
-Text Label 1900 2650 0    50   ~ 0
+Text Label 1900 2750 0    50   ~ 0
 D1-
-Text Label 1650 3000 0    50   ~ 0
+Text Label 1950 3150 0    50   ~ 0
 D2+
-Text Label 1650 3300 0    50   ~ 0
+Text Label 1950 3250 0    50   ~ 0
 D2-
 Text Label 1950 3450 0    50   ~ 0
@@
 	1800 3300 1950 3300
 Wire Wire Line
-	1900 2550 2050 2550
-Wire Wire Line
-	1900 2650 2000 2650
-Wire Wire Line
 	6050 4150 8450 4150
 Wire Wire Line
@@
 	1950 3150 2100 3150
 Wire Wire Line
-	2050 2850 2050 2550
-Wire Wire Line
-	2000 2650 2000 2950
+	2050 2850 2050 2450
+Wire Wire Line
+	2000 2750 2000 2950
 Wire Wire Line
 	1900 1600 2200 1600
@@
 Wire Wire Line
 	2200 5400 2350 5400
+Wire Wire Line
+	1800 2750 2000 2750
+Wire Wire Line
+	1800 2450 2050 2450
 $EndSCHEMATC

Commit message: corrected  output port labels
Connections:
- net labels added: 18, 19
- net labels removed: 16, 17
Changed lines of the file:
@@
 20
 Text Label 8450 2600 0    50   ~ 0
-17
+19
 Text Label 8450 2700 0    50   ~ 0
-16
+18
 Text Label 8450 2900 0    50   ~ 0
 10

Commit message: ena I²C text
Parts:
- U41: value MAX3485 -> MAX3032
Connections:
- net labels removed: DAC
Other:
- note added: "1-2\n3-4"
- note added: "To enable 5V I²C:"
- moved on the sheet: J91, JP21
Changed lines of the file:
@@
 L power:GND #PWR?
 U 1 1 5BE65233
-P 7900 5350
-F 0 "#PWR?" H 7900 5100 50  0001 C CNN
-F 1 "GND" H 7905 5177 50  0000 C CNN
-F 2 "" H 7900 5350 50  0001 C CNN
-F 3 "" H 7900 5350 50  0001 C CNN
-	1    7900 5350
+P 7600 5450
+F 0 "#PWR?" H 7600 5200 50  0001 C CNN
+F 1 "GND" H 7605 5277 50  0000 C CNN
+F 2 "" H 7600 5450 50  0001 C CNN
+F 3 "" H 7600 5450 50  0001 C CNN
+	1    7600 5450
 	1    0    0    -1
 $EndComp
@@
 P 2600 3350
 F 0 "U41" H 2950 2600 50  0000 C CNN
-F 1 "MAX3485" H 2350 2600 50  0000 C CNN
+F 1 "MAX3032" H 2350 2600 50  0000 C CNN
 F 2 "Package_SO:SOIC-16_3.9x9.9mm_P1.27mm" H 2600 2650 50  0001 C CNN
 F 3 "https://datasheets.maximintegrated.com/en/ds/MAX3483-MAX3491.pdf" H 2600 3400 50  0001 C CNN
@@
 L Connector_Generic:Conn_01x04 J91
 U 1 1 5DDE87BF
-P 8750 5200
-F 0 "J91" H 8700 5400 50  0000 L CNN
-F 1 "Conn_01x04" H 8830 5101 50  0001 L CNN
-F 2 "CANNode:OWN_KF141V-P4_simple" H 8750 5200 50  0001 C CNN
-F 3 "~" H 8750 5200 50  0001 C CNN
-	1    8750 5200
+P 8450 5300
+F 0 "J91" H 8400 5500 50  0000 L CNN
+F 1 "Conn_01x04" H 8530 5201 50  0001 L CNN
+F 2 "CANNode:OWN_KF141V-P4_simple" H 8450 5300 50  0001 C CNN
+F 3 "~" H 8450 5300 50  0001 C CNN
+	1    8450 5300
 	1    0    0    1
 $EndComp
@@
 L power:+5V #PWR?
 U 1 1 5DDFC32A
-P 8000 4950
-F 0 "#PWR?" H 8000 4800 50  0001 C CNN
-F 1 "+5V" H 8015 5123 50  0000 C CNN
-F 2 "" H 8000 4950 50  0001 C CNN
-F 3 "" H 8000 4950 50  0001 C CNN
-	1    8000 4950
+P 7700 5050
+F 0 "#PWR?" H 7700 4900 50  0001 C CNN
+F 1 "+5V" H 7715 5223 50  0000 C CNN
+F 2 "" H 7700 5050 50  0001 C CNN
+F 3 "" H 7700 5050 50  0001 C CNN
+	1    7700 5050
 	-1   0    0    -1
 $EndComp
@@
 L power:+12V #PWR?
 U 1 1 5DDFC381
-P 8100 4950
-F 0 "#PWR?" H 8100 4800 50  0001 C CNN
-F 1 "+12V" H 7950 5000 50  0000 C CNN
-F 2 "" H 8100 4950 50  0001 C CNN
-F 3 "" H 8100 4950 50  0001 C CNN
-	1    8100 4950
+P 7800 5050
+F 0 "#PWR?" H 7800 4900 50  0001 C CNN
+F 1 "+12V" H 7650 5100 50  0000 C CNN
+F 2 "" H 7800 5050 50  0001 C CNN
+F 3 "" H 7800 5050 50  0001 C CNN
+	1    7800 5050
 	-1   0    0    -1
 $EndComp
@@
 L power:+3.3V #PWR?
 U 1 1 5DDFC4E2
-P 7900 4950
-F 0 "#PWR?" H 7900 4800 50  0001 C CNN
-F 1 "+3.3V" H 8050 5000 50  0000 C CNN
-F 2 "" H 7900 4950 50  0001 C CNN
-F 3 "" H 7900 4950 50  0001 C CNN
-	1    7900 4950
+P 7600 5050
+F 0 "#PWR?" H 7600 4900 50  0001 C CNN
+F 1 "+3.3V" H 7750 5100 50  0000 C CNN
+F 2 "" H 7600 5050 50  0001 C CNN
+F 3 "" H 7600 5050 50  0001 C CNN
+	1    7600 5050
 	-1   0    0    -1
 $EndComp
 Wire Wire Line
-	8100 4950 8100 5000
-Wire Wire Line
-	8000 4950 8000 5100
-Wire Wire Line
-	7900 4950 7900 5200
-Wire Wire Line
-	7900 5300 7900 5350
+	7800 5050 7800 5100
+Wire Wire Line
+	7700 5050 7700 5200
+Wire Wire Line
+	7600 5050 7600 5300
+Wire Wire Line
+	7600 5400 7600 5450
 $Comp
 L power:GND #PWR?
@@
 Text Notes 8450 1950 0    50   ~ 0
 GPIO\n8Ch Relay Board
-Text Notes 7450 3700 0    50   ~ 0
+Text Notes 6450 5400 0    50   ~ 0
 DAC
 $Comp
@@
 	2100 2950 2000 2950
 Wire Wire Line
-	6750 5300 6550 5300
-Wire Wire Line
-	6050 5300 5400 5300
+	6750 5300 6450 5300
+Wire Wire Line
+	5950 5300 5400 5300
 Connection ~ 5400 5300
 Connection ~ 1800 2750
@@
 L power:PWR_FLAG #FLG?
 U 1 1 5D480012
-P 8450 4950
-F 0 "#FLG?" H 8450 5025 50  0001 C CNN
-F 1 "PWR_FLAG" H 8450 5124 50  0000 C CNN
-F 2 "" H 8450 4950 50  0001 C CNN
-F 3 "~" H 8450 4950 50  0001 C CNN
-	1    8450 4950
+P 8150 5050
+F 0 "#FLG?" H 8150 5125 50  0001 C CNN
+F 1 "PWR_FLAG" H 8150 5224 50  0000 C CNN
+F 2 "" H 8150 5050 50  0001 C CNN
+F 3 "~" H 8150 5050 50  0001 C CNN
+	1    8150 5050
 	-1   0    0    -1
 $EndComp
@@
 L power:PWR_FLAG #FLG?
 U 1 1 5D51B4BB
-P 8450 5350
-F 0 "#FLG?" H 8450 5425 50  0001 C CNN
-F 1 "PWR_FLAG" H 8450 5523 50  0000 C CNN
-F 2 "" H 8450 5350 50  0001 C CNN
-F 3 "~" H 8450 5350 50  0001 C CNN
-	1    8450 5350
+P 8150 5450
+F 0 "#FLG?" H 8150 5525 50  0001 C CNN
+F 1 "PWR_FLAG" H 8150 5623 50  0000 C CNN
+F 2 "" H 8150 5450 50  0001 C CNN
+F 3 "~" H 8150 5450 50  0001 C CNN
+	1    8150 5450
 	1    0    0    1
 $EndComp
 Wire Wire Line
-	8550 5000 8450 5000
-Wire Wire Line
-	8000 5100 8550 5100
-Wire Wire Line
-	8550 5200 7900 5200
-Wire Wire Line
-	7900 5300 8450 5300
-Wire Wire Line
-	8450 4950 8450 5000
-Connection ~ 8450 5000
-Wire Wire Line
-	8450 5000 8100 5000
-Wire Wire Line
-	8450 5350 8450 5300
-Connection ~ 8450 5300
-Wire Wire Line
-	8450 5300 8550 5300
+	8250 5100 8150 5100
+Wire Wire Line
+	7700 5200 8250 5200
+Wire Wire Line
+	8250 5300 7600 5300
+Wire Wire Line
+	7600 5400 8150 5400
+Wire Wire Line
+	8150 5050 8150 5100
+Connection ~ 8150 5100
+Wire Wire Line
+	8150 5100 7800 5100
+Wire Wire Line
+	8150 5450 8150 5400
+Connection ~ 8150 5400
+Wire Wire Line
+	8150 5400 8250 5400
 NoConn ~ 5350 1850
 $Comp
@@
 Text Label 1850 4400 0    50   ~ 0
 D4-
-Text Label 7150 3550 0    50   ~ 0
-DAC
 Text Label 1550 1500 0    50   ~ 0
 UA1-
@@
 L Connector_Generic:Conn_02x03_Odd_Even JP21
 U 1 1 5BF19790
-P 6350 5300
-F 0 "JP21" H 6400 5525 50  0000 C CNN
-F 1 "Conn_02x03_Odd_Even" H 6400 5526 50  0001 C CNN
-F 2 "Connector_PinHeader_2.54mm:PinHeader_2x03_P2.54mm_Vertical" H 6350 5300 50  0001 C CNN
-F 3 "~" H 6350 5300 50  0001 C CNN
-	1    6350 5300
+P 6250 5300
+F 0 "JP21" H 6300 5525 50  0000 C CNN
+F 1 "Conn_02x03_Odd_Even" H 6300 5526 50  0001 C CNN
+F 2 "Connector_PinHeader_2.54mm:PinHeader_2x03_P2.54mm_Vertical" H 6250 5300 50  0001 C CNN
+F 3 "~" H 6250 5300 50  0001 C CNN
+	1    6250 5300
 	-1   0    0    -1
 $EndComp
@@
 	5250 5200 5500 5200
 Wire Wire Line
-	5500 5200 6050 5200
+	5500 5200 5950 5200
 Connection ~ 5500 5200
 Wire Wire Line
-	6550 5200 6650 5200
+	6450 5200 6650 5200
 Wire Wire Line
 	6900 3600 6900 3700
 Wire Wire Line
-	7100 5400 6550 5400
+	7100 5400 6450 5400
 Wire Wire Line
 	7100 3600 7100 5400
@@
 L power:GND #PWR?
 U 1 1 5C338401
-P 6000 5450
-F 0 "#PWR?" H 6000 5200 50  0001 C CNN
-F 1 "GND" H 6005 5277 50  0001 C CNN
-F 2 "" H 6000 5450 50  0001 C CNN
-F 3 "" H 6000 5450 50  0001 C CNN
-	1    6000 5450
-	1    0    0    -1
-$EndComp
-Wire Wire Line
-	6050 5400 6000 5400
-Wire Wire Line
-	6000 5400 6000 5450
+P 5900 5450
+F 0 "#PWR?" H 5900 5200 50  0001 C CNN
+F 1 "GND" H 5905 5277 50  0001 C CNN
+F 2 "" H 5900 5450 50  0001 C CNN
+F 3 "" H 5900 5450 50  0001 C CNN
+	1    5900 5450
+	1    0    0    -1
+$EndComp
+Wire Wire Line
+	5950 5400 5900 5400
+Wire Wire Line
+	5900 5400 5900 5450
 $Comp
 L Device:CP_Small C11
@@
 Wire Wire Line
 	1800 2450 2050 2450
+Text Notes 5900 4800 0    50   ~ 0
+To enable 5V I²C:
+Text Notes 6100 5000 0    50   ~ 0
+1-2\n3-4
 $EndSCHEMATC

Commit message: First current messurement attempts
Parts:
- removed C1, C11, C12, C2: CP, Capacitor_SMD:CP_Elec_3x5.4, symbol Device:CP_Small
- removed U91: LM1117-5.0, Package_TO_SOT_SMD:SOT-223-3_TabPin2, symbol Regulator_Linear:LM1117-5.0
- added C10, C11, C12: 100n, Capacitor_SMD:C_0805_2012Metric_Pad1.15x1.40mm_HandSolder, symbol Device:C_Small
- added C9: C, Capacitor_SMD:C_0805_2012Metric_Pad1.15x1.40mm_HandSolder, symbol Device:C_Small
- added R12, R17, R20: 0R1, Resistor_SMD:R_2512_6332Metric, symbol Device:R_Small
- added R15, R16, R18, R19, R21, R22: 10, Resistor_SMD:R_0805_2012Metric_Pad1.15x1.40mm_HandSolder, symbol Device:R_Small
- added U6: INA3221, Package_DFN_QFN:QFN-16-1EP_4x4mm_P0.65mm_EP2.1x2.1mm, symbol JS_IC:INA3221
- MOD1: symbol 000_my_lib:DSN-MINI-360 -> CANNode-rescue:DSN-MINI-360-000_my_lib
- U3: renamed from U1; symbol teensy:Teensy3.2 -> CANNode-rescue:Teensy3.2-teensy
- U4: renamed from U41; symbol 000_my_lib:MAX3032 -> CANNode-rescue:MAX3032-000_my_lib
- renumbered C3 to C1, C4 to C2, C5 to C3, C6 to C4, C7 to C5, C8 to C6, C9 to C7, C10 to C8, J12 to J10, J44 to J11, J21 to J12, J91 to J13, J31 to J3, J81 to J4, J41 to J5, J61 to J6, J42 to J7, J11 to J8, J43 to J9, JP31 to JP1, JP1 to JP2, JP41 to JP3, JP21 to JP4, R6 to R1, R24 to R10, R25 to R11, R22 to R13, R21 to R14, R1 to R2, R2 to R3, R11 to R5, R12 to R6, R3 to R7, R5 to R8, R23 to R9, U31 to U1, U21 to U5
Connections:
- net labels added: +12L, +12LF, +5P
- wire segments 370 -> 434
Other:
- moved on the sheet: R5, R6
