File: Hardware/kicad/CANNode.sch (KiCad schematic (older format))
At the start: 48 parts, among them J1 Conn_01x04, J2 Conn_01x04, J3 Conn_01x10, J4 Conn_02x04_Odd_Even, J5 Conn_01x04, J6 Conn_01x04, J7 Conn_01x04, J8 Conn_01x03, J9 Conn_01x04, U1 MAX3485, U2 SN65HVD230, U3 Teensy3.2, U4 MAX3485, U5 PCA9306

Commit message: PCB fixed silkscreen
Parts:
- H1, H2, H3, H4: footprint MountingHole:MountingHole_3.5mm -> MountingHole:MountingHole_2.7mm
Other:
- moved on the sheet: H1, H2, H3, H4
Changed lines of the file:
@@
 Sheet 1 1
 Title "CANNode"
-Date "2018-11-17"
-Rev "2.0"
-Comp "(c) wiebel@wiebel.org"
+Date "2021-02-18"
+Rev "2.5"
+Comp "(c) mail@wiebel.org"
 Comment1 "OSH License TBD"
 Comment2 "I2C(3V3+5V), SPI"
@@
 L 00_mylib:OWN_DCDC-CANNode MOD1
 U 1 1 5BE5A42C
-P 4200 6550
-F 0 "MOD1" H 4200 6550 45  0001 C CNN
-F 1 "DSN-MINI-360" H 4200 6550 45  0001 C CNN
-F 2 "00_mylib:OWN_DC-DC" H 4200 6550 50  0001 C CNN
-F 3 "" H 4200 6550 50  0001 C CNN
-F 4 "DSN-MINI-36  (LM2596)" H 4200 6550 50  0001 C CNN "Name"
-	1    4200 6550
+P 1950 5050
+F 0 "MOD1" H 1950 5050 45  0001 C CNN
+F 1 "DSN-MINI-360" H 1950 5050 45  0001 C CNN
+F 2 "00_mylib:OWN_DC-DC" H 1950 5050 50  0001 C CNN
+F 3 "" H 1950 5050 50  0001 C CNN
+F 4 "DSN-MINI-36  (LM2596)" H 1950 5050 50  0001 C CNN "Name"
+	1    1950 5050
 	1    0    0    -1
 $EndComp
@@
 L power:+12V #PWR042
 U 1 1 5BE6267F
-P 3750 6350
-F 0 "#PWR042" H 3750 6200 50  0001 C CNN
-F 1 "+12V" H 3765 6523 50  0000 C CNN
-F 2 "" H 3750 6350 50  0001 C CNN
-F 3 "" H 3750 6350 50  0001 C CNN
-	1    3750 6350
+P 1500 4850
+F 0 "#PWR042" H 1500 4700 50  0001 C CNN
+F 1 "+12V" H 1515 5023 50  0000 C CNN
+F 2 "" H 1500 4850 50  0001 C CNN
+F 3 "" H 1500 4850 50  0001 C CNN
+	1    1500 4850
 	1    0    0    -1
 $EndComp
@@
 L power:+5V #PWR043
 U 1 1 5BE62D68
-P 4650 6350
-F 0 "#PWR043" H 4650 6200 50  0001 C CNN
-F 1 "+5V" H 4665 6523 50  0000 C CNN
-F 2 "" H 4650 6350 50  0001 C CNN
-F 3 "" H 4650 6350 50  0001 C CNN
-	1    4650 6350
+P 2400 4850
+F 0 "#PWR043" H 2400 4700 50  0001 C CNN
+F 1 "+5V" H 2415 5023 50  0000 C CNN
+F 2 "" H 2400 4850 50  0001 C CNN
+F 3 "" H 2400 4850 50  0001 C CNN
+	1    2400 4850
 	1    0    0    -1
 $EndComp
@@
 $EndComp
 Wire Wire Line
-	3750 6450 3750 6350
-Wire Wire Line
-	4650 6450 4650 6350
+	1500 4950 1500 4850
+Wire Wire Line
+	2400 4950 2400 4850
 $Comp
 L power:+5V #PWR02
@@
 	5900 5400 5900 5450
 Wire Wire Line
-	3750 6450 3800 6450
+	1500 4950 1550 4950
 Text Notes 5900 4800 0    50   ~ 0
 To enable 5V I²C:
@@
 L power:GND #PWR044
 U 1 1 5E725650
-P 4200 6850
-F 0 "#PWR044" H 4200 6600 50  0001 C CNN
-F 1 "GND" H 4205 6677 50  0000 C CNN
-F 2 "" H 4200 6850 50  0001 C CNN
-F 3 "" H 4200 6850 50  0001 C CNN
-	1    4200 6850
-	1    0    0    -1
-$EndComp
-Wire Wire Line
-	4200 6800 4200 6850
+P 1950 5350
+F 0 "#PWR044" H 1950 5100 50  0001 C CNN
+F 1 "GND" H 1955 5177 50  0000 C CNN
+F 2 "" H 1950 5350 50  0001 C CNN
+F 3 "" H 1950 5350 50  0001 C CNN
+	1    1950 5350
+	1    0    0    -1
+$EndComp
+Wire Wire Line
+	1950 5300 1950 5350
 Wire Wire Line
 	6000 2700 6100 2700
@@
 $EndComp
 Wire Wire Line
-	4600 6450 4650 6450
-Wire Wire Line
-	4600 6650 4600 6800
-Wire Wire Line
-	4600 6800 4200 6800
-Wire Wire Line
-	3800 6650 3800 6800
-Wire Wire Line
-	3800 6800 4200 6800
-Connection ~ 4200 6800
+	2350 4950 2400 4950
+Wire Wire Line
+	2350 5150 2350 5300
+Wire Wire Line
+	2350 5300 1950 5300
+Wire Wire Line
+	1550 5150 1550 5300
+Wire Wire Line
+	1550 5300 1950 5300
+Connection ~ 1950 5300
 Wire Wire Line
 	7200 950  7500 950
@@
 L 00_mylib:Logo Log1
 U 1 1 5F799D59
-P 1100 4200
-F 0 "Log1" H 1100 4200 50  0001 C CNN
-F 1 "Logo" H 1125 4200 50  0000 L CNN
-F 2 "00_mylib:LOGO_MID" H 1100 4200 50  0001 C CNN
-F 3 "" H 1100 4200 50  0001 C CNN
-	1    1100 4200
+P 650 6000
+F 0 "Log1" H 650 6000 50  0001 C CNN
+F 1 "Logo" H 675 6000 50  0000 L CNN
+F 2 "00_mylib:LOGO_MID" H 650 6000 50  0001 C CNN
+F 3 "" H 650 6000 50  0001 C CNN
+	1    650  6000
 	1    0    0    -1
 $EndComp
@@
 L 00_mylib:Logo Log2
 U 1 1 5F79ABF6
-P 1100 4300
-F 0 "Log2" H 1100 4300 50  0001 C CNN
-F 1 "Logo" H 1125 4300 50  0000 L CNN
-F 2 "Symbol:OSHW-Logo_5.7x6mm_Copper" H 1100 4300 50  0001 C CNN
-F 3 "" H 1100 4300 50  0001 C CNN
-	1    1100 4300
+P 650 6100
+F 0 "Log2" H 650 6100 50  0001 C CNN
+F 1 "Logo" H 675 6100 50  0000 L CNN
+F 2 "Symbol:OSHW-Logo_5.7x6mm_Copper" H 650 6100 50  0001 C CNN
+F 3 "" H 650 6100 50  0001 C CNN
+	1    650  6100
 	1    0    0    -1
 $EndComp
@@
 L 00_mylib:Logo Log3
 U 1 1 5F7D4FEA
-P 1100 4400
-F 0 "Log3" H 1100 4400 50  0001 C CNN
-F 1 "Logo" H 1125 4400 50  0000 L CNN
-F 2 "00_mylib:LOGO_MID" H 1100 4400 50  0001 C CNN
-F 3 "" H 1100 4400 50  0001 C CNN
-	1    1100 4400
+P 650 6200
+F 0 "Log3" H 650 6200 50  0001 C CNN
+F 1 "Logo" H 675 6200 50  0000 L CNN
+F 2 "00_mylib:LOGO_MID" H 650 6200 50  0001 C CNN
+F 3 "" H 650 6200 50  0001 C CNN
+	1    650  6200
 	1    0    0    -1
 $EndComp
@@
 L 00_mylib:Logo Log4
 U 1 1 5F7D4FF0
-P 1100 4500
-F 0 "Log4" H 1100 4500 50  0001 C CNN
-F 1 "Logo" H 1125 4500 50  0000 L CNN
-F 2 "Symbol:OSHW-Logo_5.7x6mm_Copper" H 1100 4500 50  0001 C CNN
-F 3 "" H 1100 4500 50  0001 C CNN
-	1    1100 4500
+P 650 6300
+F 0 "Log4" H 650 6300 50  0001 C CNN
+F 1 "Logo" H 675 6300 50  0000 L CNN
+F 2 "Symbol:OSHW-Logo_5.7x6mm_Copper" H 650 6300 50  0001 C CNN
+F 3 "" H 650 6300 50  0001 C CNN
+	1    650  6300
 	1    0    0    -1
 $EndComp
@@
 L Mechanical:MountingHole H1
 U 1 1 5F8345AF
-P 1200 4750
-F 0 "H1" H 1300 4796 50  0000 L CNN
-F 1 "MountingHole" H 1300 4705 50  0000 L CNN
-F 2 "MountingHole:MountingHole_3.5mm" H 1200 4750 50  0001 C CNN
-F 3 "~" H 1200 4750 50  0001 C CNN
-	1    1200 4750
+P 750 6550
+F 0 "H1" H 850 6596 50  0000 L CNN
+F 1 "MountingHole" H 850 6505 50  0000 L CNN
+F 2 "MountingHole:MountingHole_2.7mm" H 750 6550 50  0001 C CNN
+F 3 "~" H 750 6550 50  0001 C CNN
+	1    750  6550
 	1    0    0    -1
 $EndComp
@@
 L Mechanical:MountingHole H2
 U 1 1 5F834FEC
-P 1200 4950
-F 0 "H2" H 1300 4996 50  0000 L CNN
-F 1 "MountingHole" H 1300 4905 50  0000 L CNN
-F 2 "MountingHole:MountingHole_3.5mm" H 1200 4950 50  0001 C CNN
-F 3 "~" H 1200 4950 50  0001 C CNN
-	1    1200 4950
+P 750 6750
+F 0 "H2" H 850 6796 50  0000 L CNN
+F 1 "MountingHole" H 850 6705 50  0000 L CNN
+F 2 "MountingHole:MountingHole_2.7mm" H 750 6750 50  0001 C CNN
+F 3 "~" H 750 6750 50  0001 C CNN
+	1    750  6750
 	1    0    0    -1
 $EndComp
@@
 L Mechanical:MountingHole H3
 U 1 1 5F84F730
-P 1200 5150
-F 0 "H3" H 1300 5196 50  0000 L CNN
-F 1 "MountingHole" H 1300 5105 50  0000 L CNN
-F 2 "MountingHole:MountingHole_3.5mm" H 1200 5150 50  0001 C CNN
-F 3 "~" H 1200 5150 50  0001 C CNN
-	1    1200 5150
+P 750 6950
+F 0 "H3" H 850 6996 50  0000 L CNN
+F 1 "MountingHole" H 850 6905 50  0000 L CNN
+F 2 "MountingHole:MountingHole_2.7mm" H 750 6950 50  0001 C CNN
+F 3 "~" H 750 6950 50  0001 C CNN
+	1    750  6950
 	1    0    0    -1
 $EndComp
@@
 L Mechanical:MountingHole H4
 U 1 1 5F869DBA
-P 1200 5350
-F 0 "H4" H 1300 5396 50  0000 L CNN
-F 1 "MountingHole" H 1300 5305 50  0000 L CNN
-F 2 "MountingHole:MountingHole_3.5mm" H 1200 5350 50  0001 C CNN
-F 3 "~" H 1200 5350 50  0001 C CNN
-	1    1200 5350
-	1    0    0    -1
-$EndComp
+P 750 7150
+F 0 "H4" H 850 7196 50  0000 L CNN
+F 1 "MountingHole" H 850 7105 50  0000 L CNN
+F 2 "MountingHole:MountingHole_2.7mm" H 750 7150 50  0001 C CNN
+F 3 "~" H 750 7150 50  0001 C CNN
+	1    750  7150
+	1    0    0    -1
+$EndComp
